File: PCB Design/JakesPad/JakesPad.kicad_pcb (KiCad board)
At the start: 2 copper layers, 277 x 171 mm, 39 parts, among them SW1 SW_Push, SW2 SW_Push, SW3 SW_Push, SW4 SW_Push, SW5 SW_Push, SW6 SW_Push, U2 rp2040-zero

Commit message: Big Update
Parts:
- SW1, SW2, SW3, SW4, SW5, SW6: footprint Button_Switch_THT:SW_PUSH-12mm -> RanilCustom:SW_PUSH-12mmWithCAD
Other:
- board text added: "Jake's Pad (Custom GamePad Controller) REV: 0.2 Name: Ranil Ganlath Date: 02-28-2024 S/N:"
- board text removed: "Jake's Pad (Custom GamePad Controller) REV: 0.1 Name: Ranil Ganlath Date: 02-21-2024 S/N:"
